File: Hardware/Qwiic_UV_Sensor_VEML6075.brd (EAGLE design)
At the start: 25.4 x 25.4 mm, 35 parts, among them J3 PTH, U1 VEML6075

Commit message: post checklist changes
Parts:
- U1: device Qwiic_UV_Sensor_VEML6075:VEML6075_A3OP -> SparkFun-Sensors:VEML6075_A3OP
