File: Hardware/Qwiic_UV_Sensor_VEML6075.sch (EAGLE design)
At the start: 21 parts, among them J3 PTH, U1 VEML6075

Commit message: post checklist changes
Parts:
- U1: device Qwiic_UV_Sensor_VEML6075:VEML6075 -> SparkFun-Sensors:VEML6075
Other:
- note added: "Disconnect jumper JP1 to disconnect the I2C pullup resistors. Do this if you have many boards on a bus to save on power consumption."
Changed lines of the file:
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@@
 <parts>
 <part name="FRAME1" library="SparkFun-Aesthetics" deviceset="FRAME-LETTER" device=""/>
-<part name="U1" library="Qwiic_UV_Sensor_VEML6075" deviceset="VEML6075" device=""/>
+<part name="U1" library="SparkFun-Sensors" deviceset="VEML6075" device=""/>
 <part name="R3" library="SparkFun-Resistors" deviceset="1KOHM" device="-0603-1/10W-1%" value="1k"/>
 <part name="SUPPLY10" library="SparkFun-PowerSymbols" deviceset="3.3V" device=""/>
@@
 <text x="168.656" y="7.112" size="2.54" layer="94" font="vector">Andy England</text>
 <text x="121.92" y="157.48" size="2.54" layer="97" font="vector">Vin: 1.7-3.6V</text>
+<text x="160.02" y="147.32" size="1.778" layer="97" font="vector">Disconnect jumper JP1 to disconnect
+the I2C pullup resistors. Do this if you
+have many boards on a bus to save on
+power consumption.</text>
 </plain>
 <instances>
@@
 <instance part="LOGO1" gate="G$1" x="45.72" y="12.7"/>
 <instance part="U$1" gate="G$1" x="58.42" y="2.54"/>
-<instance part="JP3" gate="G$1" x="246.38" y="30.48"/>
-<instance part="JP4" gate="G$1" x="246.38" y="27.94"/>
+<instance part="JP3" gate="G$1" x="238.76" y="30.48"/>
+<instance part="JP4" gate="G$1" x="238.76" y="27.94"/>
 <instance part="JP2" gate="G$1" x="233.68" y="30.48"/>
 <instance part="JP6" gate="G$1" x="236.22" y="30.48"/>
@@
 </schematic>
 </drawing>
+<compatibility>
+<note version="6.3" minversion="6.2.2" severity="warning">
+Since Version 6.2.2 text objects can contain more than one line,
+which will not be processed correctly with this version.
+</note>
+</compatibility>
 </eagle>
